File: BLDC_driver_small.kicad_sch (KiCad schematic)
At the start: 33 parts

Commit message: 120323
Parts:
- removed C?: 100n, symbol Device:C_Small
- removed C?: ?, symbol Device:C_Small
- removed C?: Cx, symbol Device:C_Small
- removed R?: R1, symbol Device:R_Small
- removed R? (x2): Rfbk, symbol Device:R_Small
- removed R? (x2): Rin, symbol Device:R_Small
- removed R?: R2, symbol Device:R_Small
- removed R? (x2): ?R, symbol Device:R_Small
- removed R?: Rx, symbol Device:R_Small
- removed U? (x3): Opamp_Quad, symbol Device:Opamp_Quad
- removed U?: STM32G030F6Px, Package_SO:TSSOP-20_4.4x6.5mm_P0.65mm, symbol fraciscoestar:STM32G030F6Px
- added C? (x3): 1n, symbol Device:C_Small
- added C? (x3): 100n, symbol Device:C_Small
- added D?: 24V, symbol Device:D_Zener_Small
- added F?: Polyfuse, symbol Device:Polyfuse_Small
- added Q?: Q_PMOS_GDS, symbol Device:Q_PMOS_GDS
- added R? (x6): 1M, symbol Device:R_Small
- added R?: 10k, symbol Device:R_Small
- added SW?: SW_SPDT, symbol Switch:SW_SPDT
- added SW?: RST_SW, symbol Switch:SW_Push_45deg
- added U?: STM32F030K6Tx, Package_QFP:LQFP-32_7x7mm_P0.8mm, symbol MCU_ST_STM32F0:STM32F030K6Tx
- J?: value Screw_Terminal_01x02 -> 1x02 Terminal
- J?: value Screw_Terminal_01x03 -> 1x03 Terminal
- R? (x3): value 1R -> 10m
Connections:
- net ~{ADC_{ENABLE}} is gone; now on net GND: U?.12 (~{CS})
- net +24V: now also C?.1, C?.1, D?.1 (K), Q?.3 (S); no longer J?.1 (Pin_1)
- net +3.3VA: now also U?.5 (VDDA)
- net +3V3: now also SW?.1 (A), U?.1 (VDD), U?.17 (VDD)
- net ADC_{CLKIN}: now also U?.18 (PA8)
- net ADC_{IN0}+: now also C?.1, R?.2
- net ADC_{IN0}-: now also C?.2, R?.2
- net ADC_{IN1}+: now also C?.1, R?.2
- net ADC_{IN1}-: now also C?.2, R?.2
- net ADC_{IN2}+: now also C?.1, R?.2
- net ADC_{IN2}-: now also C?.2, R?.2
- net ADC_{MISO}: now also U?.12 (PA6)
- net ADC_{MOSI}: now also U?.13 (PA7)
- net ADC_{SCLK}: now also U?.11 (PA5)
- net GND: now also C?.2, C?.2, C?.2, SW?.1, SW?.3 (C), U?.16 (VSS), U?.32 (VSS); no longer C?.2
- net GNDA: now also C?.2; no longer C?.2, J?.2 (Pin_2), R?.2, R?.2, R?.2
- net PWM_{U}: now also U?.21 (PA11)
- net PWM_{V}: now also U?.20 (PA10)
- net PWM_{W}: now also U?.19 (PA9)
- net ~{ADC_{DRDY}}: now also U?.10 (PA4)
- net ~{ADC_{RST}}: now also U?.14 (PB0)
- net at U?.24 (VCP): now also C?.2
- net +1V2: now reaches C?.1, U?.18 (CAP)
- net SENSE_{U} renamed SENSE_{U}+
- net SENSE_{U}+: now also R?.1
- net SENSE_{V} renamed SENSE_{V}+
- net SENSE_{V}+: now also R?.1
- net SENSE_{W} renamed SENSE_{W}+
- net SENSE_{W}+: now also R?.1
- new net: SW?.2 (B), U?.31 (BOOT0)
- new net: F?.1, J?.1 (Pin_1)
- new net: F?.2, Q?.2 (D)
- new net: D?.2 (A), Q?.1 (G), R?.2
- new net GNDPWR: C?.2, J?.2 (Pin_2), R?.1, R?.1, R?.1, R?.1, R?.2, R?.2, R?.2
- new net I2C_{SCL}: U?.29 (PB6)
- new net I2C_{SDA}: U?.30 (PB7)
- new net NRST: C?.1, SW?.2, U?.4 (NRST)
- new net SWD_{CLK}: U?.24 (PA14)
- new net SWD_{IO}: U?.23 (PA13)
- new net UART_{RX}: U?.9 (PA3)
- new net UART_{TX}: U?.8 (PA2)
Other:
- note removed: "V_{offset}=R_{2}/(R_{1}+R_{2}) V_{out}=(I_{DC}*R_{shunt})*(R_{fbk}/R_{in})+V_{offset}"
- moved on the sheet: C?, D?, J?, R?, U?

Commit message: 120223-2
Parts:
- removed U?: ADS131M03IPWR, Package_SO:TSSOP-20_4.4x6.5mm_P0.65mm, symbol fraciscoestar:ADS131M03IPWR
- added C1, C2: 1u, Capacitor_SMD:C_0603_1608Metric, symbol Device:C_Small
- added C10, C8, C9: 100n, Capacitor_SMD:C_0402_1005Metric, symbol Device:C_Small
- added C18, C19: TBD, Capacitor_SMD:C_0402_1005Metric, symbol Device:C_Small
- added C3: 10n, Capacitor_SMD:C_0603_1608Metric, symbol Device:C_Small
- added C5: 2u2, Capacitor_SMD:C_0805_2012Metric, symbol Device:C_Small
- added C6, C7: 4u7, Capacitor_SMD:C_0603_1608Metric, symbol Device:C_Small
- added L1: 10u, Inductor_SMD:L_6.3x6.3_H3, symbol Device:L_Small
- added L2: 39n, Inductor_SMD:L_0603_1608Metric, symbol Device:L_Small
- added R1: 806k, Resistor_SMD:R_0603_1608Metric, symbol Device:R_Small
- added R11: 47R, Resistor_SMD:R_0603_1608Metric, symbol Device:R_Small
- added R3: 500k, Resistor_SMD:R_0603_1608Metric, symbol Device:R_Small
- added R6: 10k, Resistor_SMD:R_0603_1608Metric, symbol Device:R_Small
- added U1: NCP786L, Package_TO_SOT_SMD:SOT-223, symbol fraciscoestar:NCP786L
- added U3: ADS131M03IPWR, Package_SO:TSSOP-20_4.4x6.5mm_P0.65mm, symbol fraciscoestar:ADS131M03IPWR
- added Y1: 16MHz, Crystal:Crystal_SMD_3225-4Pin_3.2x2.5mm, symbol Device:Crystal_GND24_Small
- C11, C12, C21, C23, C24: renamed from C?; footprint (none) -> Capacitor_SMD:C_0603_1608Metric
- C13, C14, C15, C16, C17, C20, C22: renamed from C?; footprint (none) -> Capacitor_SMD:C_0402_1005Metric
- C4: renamed from C?; footprint (none) -> Capacitor_SMD:CP_Elec_6.3x5.4
- D1: renamed from D?; footprint (none) -> Diode_SMD:D_SOD-123
- D2, D3: renamed from D?; footprint (none) -> Diode_SMD:D_SOD-323
- J1: renamed from J?; footprint (none) -> TerminalBlock:TerminalBlock_Altech_AK300-2_P5.00mm
- J2: renamed from J?; footprint (none) -> TerminalBlock:TerminalBlock_Altech_AK300-3_P5.00mm
- Q1: renamed from Q?; footprint (none) -> Package_TO_SOT_SMD:SOT-23
- R10, R12, R13, R14, R15, R2, R4, R8: renamed from R?; footprint (none) -> Resistor_SMD:R_0603_1608Metric
- R5, R7, R9: renamed from R?; footprint (none) -> Resistor_SMD:R_1210_3225Metric
- SW1: renamed from SW?; footprint (none) -> Button_Switch_SMD:SW_SPST_B3S-1000
- SW2: renamed from SW?; footprint (none) -> Button_Switch_SMD:SW_SPDT_PCM12
- gave numbers to parts that had none: 3
Connections:
- net GNDA is gone; now on net GND: C14.2, C23.2
- net GNDPWR is gone; now on net GND: C4.2, J1.2 (Pin_2), R12.1, R15.1, R2.1, R5.2, R7.2, R8.1, R9.2
- net +1V2: now also U3.18 (CAP)
- net +24V: now also C5.1, L1.2, U1.1 (VIN); no longer D1.1 (K), Q1.3 (S)
- net +3.3VA: now also C10.1, C2.1, C3.1, L2.2, U3.1 (AVDD)
- net +3V3: now also C1.1, C6.1, C7.1, C8.1, C9.1, L2.1, R1.2, U1.3 (VOUT), U3.20 (DVDD)
- net ADC_{CLKIN}: now also U3.17 (CLKIN)
- net ADC_{IN0}+: now also U3.3 (AIN0P)
- net ADC_{IN0}-: now also U3.4 (AIN0N)
- net ADC_{IN1}+: now also U3.6 (AIN1P)
- net ADC_{IN1}-: now also U3.5 (AIN1N)
- net ADC_{IN2}+: now also U3.7 (AIN2P)
- net ADC_{IN2}-: now also U3.8 (AIN2N)
- net ADC_{MISO}: now also U3.15 (DOUT)
- net ADC_{MOSI}: now also U3.16 (DIN)
- net ADC_{SCLK}: now also U3.14 (SCLK)
- net ENA_{U}: now also U4.26 (PB3)
- net ENA_{V}: now also U4.27 (PB4)
- net ENA_{W}: now also U4.28 (PB5)
- net GND: now also C1.2, C10.2, C18.2, C19.2, C2.2, C3.2, C5.2, C6.2, C7.2, C8.2, C9.2, R3.1, U1.4 (GND), U3.12 (~{CS}), U3.19 (DGND), U3.2 (AGND), Y1.2, Y1.4
- net ~{ADC_{DRDY}}: now also U3.13 (~{DRDY})
- net ~{ADC_{RST}}: now also U3.11 (~{SYNC}/~{RESET})
- net at SW2.2 (B): now also R6.1; no longer U4.31 (BOOT0)
- net OUT_{U}: now reaches J2.1 (Pin_1), U2.15 (OUT1)
- net at C21.2: now also U2.7 (VCP); no longer U2.24 (VCP)
- net OUT_{W}: now reaches J2.3 (Pin_3), U2.32 (OUT3)
- net OUT_{V}: now reaches J2.2 (Pin_2), U2.5 (OUT2)
- net at U4.15 (PB1): now also R14.2
- net OSC_{IN}: now reaches U4.2 (PF0)
- net OSC_{IN}: now also C19.1, Y1.1
- net at U4.3 (PF1): now also R11.2
- new net: R1.1, R3.2, U1.2 (ADJ)
- new net: R6.2, U4.31 (BOOT0)
- new net: D1.1 (K), L1.1, Q1.3 (S)
- new net OSC_{OUT}: C18.1, R11.1, Y1.3
Other:
- note added: "+3V3 = 1.27*(1+806/500) = 3.31724V"
- note removed: "PUSH-PULL signal only"
- moved on the sheet: C13, C22, C4, J2, R14, SW1, SW2

Commit message: 130323
Parts:
- C23: footprint Capacitor_SMD:C_0603_1608Metric -> Resistor_SMD:R_0402_1005Metric
- F1: footprint (none) -> Resistor_SMD:R_0805_2012Metric
- R10, R12, R13, R15, R4, R8: value 1M -> 500k; footprint Resistor_SMD:R_0603_1608Metric -> Resistor_SMD:R_0402_1005Metric
- R11: footprint Resistor_SMD:R_0603_1608Metric -> Resistor_SMD:R_0402_1005Metric
Changed lines of the file:
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@@
     (pin "23")
     (pin "24")
-    (pin "7")
     (pin "25")
     (pin "26")
@@
     (pin "5")
     (pin "6")
+    (pin "7")
     (pin "8")
     (pin "9")
@@
       (effects (font (size 1 1)))
     )
-    (property "Value" "1M" (id 1) (at 111.76 97.79 90)
-      (effects (font (size 1 1)))
-    )
-    (property "Footprint" "Resistor_SMD:R_0603_1608Metric" (id 2) (at 111.76 97.79 0)
+    (property "Value" "500k" (id 1) (at 111.76 97.79 90)
+      (effects (font (size 1 1)))
+    )
+    (property "Footprint" "Resistor_SMD:R_0402_1005Metric" (id 2) (at 111.76 97.79 0)
       (effects (font (size 1.27 1.27)) hide)
     )
@@
       (effects (font (size 1 1)))
     )
-    (property "Value" "1M" (id 1) (at 111.76 85.09 90)
-      (effects (font (size 1 1)))
-    )
-    (property "Footprint" "Resistor_SMD:R_0603_1608Metric" (id 2) (at 111.76 85.09 0)
+    (property "Value" "500k" (id 1) (at 111.76 85.09 90)
+      (effects (font (size 1 1)))
+    )
+    (property "Footprint" "Resistor_SMD:R_0402_1005Metric" (id 2) (at 111.76 85.09 0)
       (effects (font (size 1.27 1.27)) hide)
     )
@@
       (effects (font (size 1 1)))
     )
-    (property "Value" "1M" (id 1) (at 111.76 110.49 90)
-      (effects (font (size 1 1)))
-    )
-    (property "Footprint" "Resistor_SMD:R_0603_1608Metric" (id 2) (at 111.76 110.49 0)
+    (property "Value" "500k" (id 1) (at 111.76 110.49 90)
+      (effects (font (size 1 1)))
+    )
+    (property "Footprint" "Resistor_SMD:R_0402_1005Metric" (id 2) (at 111.76 110.49 0)
       (effects (font (size 1.27 1.27)) hide)
     )
@@
       (effects (font (size 1 1)))
     )
-    (property "Footprint" "" (id 2) (at 40.64 20.32 0)
+    (property "Footprint" "Resistor_SMD:R_0805_2012Metric" (id 2) (at 40.64 20.32 0)
       (effects (font (size 1.27 1.27)) (justify left) hide)
     )
@@
       (effects (font (size 1 1)))
     )
-    (property "Value" "1M" (id 1) (at 111.76 90.17 90)
-      (effects (font (size 1 1)))
-    )
-    (property "Footprint" "Resistor_SMD:R_0603_1608Metric" (id 2) (at 111.76 90.17 0)
+    (property "Value" "500k" (id 1) (at 111.76 90.17 90)
+      (effects (font (size 1 1)))
+    )
+    (property "Footprint" "Resistor_SMD:R_0402_1005Metric" (id 2) (at 111.76 90.17 0)
       (effects (font (size 1.27 1.27)) hide)
     )
@@
       (effects (font (size 1 1)))
     )
-    (property "Value" "1M" (id 1) (at 111.76 102.87 90)
-      (effects (font (size 1 1)))
-    )
-    (property "Footprint" "Resistor_SMD:R_0603_1608Metric" (id 2) (at 111.76 102.87 0)
+    (property "Value" "500k" (id 1) (at 111.76 102.87 90)
+      (effects (font (size 1 1)))
+    )
+    (property "Footprint" "Resistor_SMD:R_0402_1005Metric" (id 2) (at 111.76 102.87 0)
       (effects (font (size 1.27 1.27)) hide)
     )
@@
       (effects (font (size 1 1)) (justify left))
     )
-    (property "Footprint" "Capacitor_SMD:C_0603_1608Metric" (id 2) (at 161.29 109.22 0)
+    (property "Footprint" "Resistor_SMD:R_0402_1005Metric" (id 2) (at 161.29 109.22 0)
       (effects (font (size 1.27 1.27)) hide)
     )
@@
       (effects (font (size 1 1)))
     )
-    (property "Value" "1M" (id 1) (at 111.76 77.47 90)
-      (effects (font (size 1 1)))
-    )
-    (property "Footprint" "Resistor_SMD:R_0603_1608Metric" (id 2) (at 111.76 77.47 0)
+    (property "Value" "500k" (id 1) (at 111.76 77.47 90)
+      (effects (font (size 1 1)))
+    )
+    (property "Footprint" "Resistor_SMD:R_0402_1005Metric" (id 2) (at 111.76 77.47 0)
       (effects (font (size 1.27 1.27)) hide)
     )
@@
       (effects (font (size 1 1)))
     )
-    (property "Footprint" "Resistor_SMD:R_0603_1608Metric" (id 2) (at 219.71 95.25 0)
+    (property "Footprint" "Resistor_SMD:R_0402_1005Metric" (id 2) (at 219.71 95.25 0)
       (effects (font (size 1.27 1.27)) hide)
     )
@@
     )
     (path "/b40a4e60-049c-4958-8c1f-bfacc3465d54"
-      (reference "C23") (unit 1) (value "220n") (footprint "Capacitor_SMD:C_0603_1608Metric")
+      (reference "C23") (unit 1) (value "220n") (footprint "Resistor_SMD:R_0402_1005Metric")
     )
     (path "/56352059-2465-4e61-bda1-e6890d343ade"
@@
     )
     (path "/90527624-b5c2-4f05-ad01-a7fbd4efe8c3"
-      (reference "F1") (unit 1) (value "Polyfuse") (footprint "")
+      (reference "F1") (unit 1) (value "Polyfuse") (footprint "Resistor_SMD:R_0805_2012Metric")
     )
     (path "/3a1a15bf-aca9-41db-abbd-367c8fae8ee8"
@@
     )
     (path "/b6526dea-bcfa-4aa0-a297-323ce4603cfa"
-      (reference "R4") (unit 1) (value "1M") (footprint "Resistor_SMD:R_0603_1608Metric")
+      (reference "R4") (unit 1) (value "500k") (footprint "Resistor_SMD:R_0402_1005Metric")
     )
     (path "/744db069-3cf9-445c-b41b-bf2ce4ebae84"
@@
     )
     (path "/3ee71806-d2cd-4685-8afa-83ee586e8123"
-      (reference "R8") (unit 1) (value "1M") (footprint "Resistor_SMD:R_0603_1608Metric")
+      (reference "R8") (unit 1) (value "500k") (footprint "Resistor_SMD:R_0402_1005Metric")
     )
     (path "/901adbdb-a84d-4575-8597-0ece54a92b22"
@@
     )
     (path "/a726821c-57c2-4f69-9200-05f1678ebc59"
-      (reference "R10") (unit 1) (value "1M") (footprint "Resistor_SMD:R_0603_1608Metric")
+      (reference "R10") (unit 1) (value "500k") (footprint "Resistor_SMD:R_0402_1005Metric")
     )
     (path "/dcfff382-6f8f-42c3-8be9-2c7a1c352836"
-      (reference "R11") (unit 1) (value "47R") (footprint "Resistor_SMD:R_0603_1608Metric")
+      (reference "R11") (unit 1) (value "47R") (footprint "Resistor_SMD:R_0402_1005Metric")
     )
     (path "/36466316-4053-450f-8723-f3c4d652746b"
-      (reference "R12") (unit 1) (value "1M") (footprint "Resistor_SMD:R_0603_1608Metric")
+      (reference "R12") (unit 1) (value "500k") (footprint "Resistor_SMD:R_0402_1005Metric")
     )
     (path "/ad87c23a-abe0-4ba4-9b03-542477d03dbf"
-      (reference "R13") (unit 1) (value "1M") (footprint "Resistor_SMD:R_0603_1608Metric")
+      (reference "R13") (unit 1) (value "500k") (footprint "Resistor_SMD:R_0402_1005Metric")
     )
     (path "/71a425d8-cc32-4feb-a8a5-65876e946ad4"
@@
     )
     (path "/8cf80a87-44ea-4a83-8c56-b13f41c49718"
-      (reference "R15") (unit 1) (value "1M") (footprint "Resistor_SMD:R_0603_1608Metric")
+      (reference "R15") (unit 1) (value "500k") (footprint "Resistor_SMD:R_0402_1005Metric")
     )
     (path "/5dd67c1b-50f9-45d6-b6ef-a9b2942eec2a"

Commit message: 130323-2
Parts:
- removed U2: L6230PD, fraciscoestar:PowerSO36, symbol fraciscoestar:L6230PD
- added R? (x3): 39k, Resistor_SMD:R_0603_1608Metric, symbol Device:R_Small
- added U2: L6230Q, fraciscoestar:VFQFPN32, symbol fraciscoestar:L6230Q
- C4: footprint Capacitor_SMD:CP_Elec_6.3x5.4 -> Capacitor_SMD:CP_Elec_10x12.5
- R5, R7, R9: value 10m -> 0.33
Connections:
- net +24V: now also U2.20 (VSB), U2.22 (VSA)
- net ENA_{DRV}: now also U2.9 (DIAG-EN)
- net ENA_{U}: now also R?.2, U2.27 (EN1)
- net ENA_{V}: now also R?.2, R?.2, U2.14 (EN2)
- net ENA_{W}: now also U2.16 (EN3)
- net GND: now also R?.1, R?.1, R?.1, U2.1 (GND), U2.21 (GND)
- net OUT_{U}: now also U2.31 (OUT1)
- net OUT_{V}: now also U2.23 (OUT2)
- net OUT_{W}: now also U2.19 (OUT3)
- net PWM_{U}: now also U2.26 (IN1)
- net PWM_{V}: now also U2.13 (IN2)
- net PWM_{W}: now also U2.28 (IN3)
- net SENSE_{U}+: now also U2.29 (SENSE1)
- net SENSE_{V}+: now also U2.25 (SENSE2)
- net SENSE_{W}+: now also U2.12 (SENSE3)
- net V_{BOOT}: now also U2.17 (VBOOT)
- net at C21.2: now also U2.24 (VCP)
- net at U4.15 (PB1): no longer R14.2
Other:
- moved on the sheet: C18, C19, C22, R14, Y1

Commit message: 130323-3 fullchange
Parts:
- removed C10, C13, C8, C9: 100n, Capacitor_SMD:C_0402_1005Metric, symbol Device:C_Small
- removed C14, C15: 1u, Capacitor_SMD:C_0402_1005Metric, symbol Device:C_Small
- removed C16, C17, C20: 1n, Capacitor_SMD:C_0402_1005Metric, symbol Device:C_Small
- removed C22: 5n6, Capacitor_SMD:C_0402_1005Metric, symbol Device:C_Small
- removed C23: 220n, Resistor_SMD:R_0402_1005Metric, symbol Device:C_Small
- removed C5: 2u2, Capacitor_SMD:C_0805_2012Metric, symbol Device:C_Small
- removed C6, C7: 4u7, Capacitor_SMD:C_0603_1608Metric, symbol Device:C_Small
- removed R1: 806k, Resistor_SMD:R_0603_1608Metric, symbol Device:R_Small
- removed R10, R12, R13, R15, R4, R8: 500k, Resistor_SMD:R_0402_1005Metric, symbol Device:R_Small
- removed R11: 47R, Resistor_SMD:R_0402_1005Metric, symbol Device:R_Small
- removed R14: 100k, Resistor_SMD:R_0603_1608Metric, symbol Device:R_Small
- removed R3: 500k, Resistor_SMD:R_0603_1608Metric, symbol Device:R_Small
- removed R6: 10k, Resistor_SMD:R_0603_1608Metric, symbol Device:R_Small
- removed R? (x3): 39k, Resistor_SMD:R_0603_1608Metric, symbol Device:R_Small
- removed SW1: RST_SW, Button_Switch_SMD:SW_SPST_B3S-1000, symbol Switch:SW_Push_45deg
- removed SW2: SW_SPDT, Button_Switch_SMD:SW_SPDT_PCM12, symbol Switch:SW_SPDT
- removed U1: NCP786L, Package_TO_SOT_SMD:SOT-223, symbol fraciscoestar:NCP786L
- removed U3: ADS131M03IPWR, Package_SO:TSSOP-20_4.4x6.5mm_P0.65mm, symbol fraciscoestar:ADS131M03IPWR
- removed U4: STM32F030K6Tx, Package_QFP:LQFP-32_7x7mm_P0.8mm, symbol MCU_ST_STM32F0:STM32F030K6Tx
- added C? (x5): 100n, Capacitor_SMD:C_0402_1005Metric, symbol Device:C_Small
- added C? (x3): 680p, Capacitor_SMD:C_0402_1005Metric, symbol Device:C_Small
- added C? (x3): 100p, Capacitor_SMD:C_0402_1005Metric, symbol Device:C_Small
- added C? (x3): 4u7, Capacitor_SMD:C_0603_1608Metric, symbol Device:C_Small
- added C?: 5n6, Capacitor_SMD:C_0402_1005Metric, symbol Device:C_Small
- added C?: 1u, Capacitor_SMD:C_0805_2012Metric, symbol Device:C_Small
- added D?: LED, symbol Device:LED
- added J?: Conn_01x04, symbol Connector_Generic:Conn_01x04
- added J?: Conn_02x05_Odd_Even, symbol Connector_Generic:Conn_02x05_Odd_Even
- added R? (x10): 2k2, Resistor_SMD:R_1210_3225Metric, symbol Device:R_Small
- added R? (x3): 680, Resistor_SMD:R_1210_3225Metric, symbol Device:R_Small
- added R? (x2): 10k, Resistor_SMD:R_0603_1608Metric, symbol Device:R_Small
- added R? (x3): 0R, Resistor_SMD:R_1210_3225Metric, symbol Device:R_Small
- added R?: 2k2, Resistor_SMD:R_0603_1608Metric, symbol Device:R_Small
- added R?: 47R, Resistor_SMD:R_0402_1005Metric, symbol Device:R_Small
- added R?: 100k, Resistor_SMD:R_0603_1608Metric, symbol Device:R_Small
- added SW?: SW_SPDT, Button_Switch_SMD:SW_SPDT_PCM12, symbol Switch:SW_SPDT
- added SW?: SW_Push_45deg, symbol Switch:SW_Push_45deg
- added SW?: RST_SW, Button_Switch_SMD:SW_SPST_B3S-1000, symbol Switch:SW_Push_45deg
- added U?: TLS850C2TEV33, Package_TO_SOT_SMD:TO-252-5_TabPin3, symbol fraciscoestar:TLS850C2TEV33
- added U? (x5): TSV994, symbol Amplifier_Operational:TSV994
- added U?: STM32F030F4Px, Package_SO:TSSOP-20_4.4x6.5mm_P0.65mm, symbol MCU_ST_STM32F0:STM32F030F4Px
- Y1: value 16MHz -> 48MHz
Connections:
- net ENA_{V} is gone; now on net ENABLE: U2.14 (EN2)
- net ENA_{W} is gone; now on net ENABLE: U2.16 (EN3)
- net +24V: now also C?.1, U?.1 (I)
- net +3.3VA: now also C?.1, C?.1, R?.2, R?.2, R?.2, U?.4 (V+), U?.5 (VDDA)
- net +3V3: now also C?.1, C?.1, C?.1, C?.1, J?.1 (Pin_1), J?.2 (Pin_2), R?.2, R?.2, SW?.1 (A), U?.16 (VDD), U?.5 (Q)
- net ENA_{DRV}: now also C?.1, R?.1
- net GND: now also U2.2 (NC), U2.3 (NC), U2.4 (NC), U2.5 (NC), U2.6 (NC), U2.7 (NC), U2.8 (NC), C?.1, C?.1, C?.1, C?.2, C?.2, C?.2, C?.2, C?.2, C?.2, C?.2, C?.2, C?.2, C?.2, D?.1 (K), J?.1 (Pin_1), J?.3 (Pin_3), J?.5 (Pin_5), J?.9 (Pin_9), R?.2, R?.2, R?.2, SW?.1, SW?.1, SW?.3 (C), U?.11 (V-), U?.15 (VSS), U?.3 (GND)
- net I2C_{SCL}: now also J?.3 (Pin_3), U?.17 (PA9)
- net I2C_{SDA}: now also J?.4 (Pin_4), U?.18 (PA10)
- net NRST: now also C?.1, J?.10 (Pin_10), SW?.2, U?.4 (NRST)
- net OSC_{IN}: now also U?.2 (PF0)
- net OSC_{OUT}: now also R?.1
- net PWM_{U}: now also U?.14 (PB1)
- net PWM_{V}: now also U?.12 (PA6)
- net PWM_{W}: now also U?.13 (PA7)
- net SENSE_{U}+: now also R?.2
- net SENSE_{V}+: now also R?.2
- net SENSE_{W}+: now also R?.2
- net SWD_{CLK}: now also J?.4 (Pin_4), U?.20 (PA14)
- net SWD_{IO}: now also J?.2 (Pin_2), U?.19 (PA13)
- net ENA_{U} renamed ENABLE
- net ENABLE: now also R?.2, U?.11 (PA5)
- new net: C?.2, R?.1, R?.2, U?.7
- new net: C?.1, R?.1, R?.2, U?.6 (-)
- new net: C?.2, R?.1, R?.1, U?.3 (+)
- new net: C?.2, R?.1, R?.2, U?.1
- new net: C?.1, R?.1, R?.2, U?.2 (-)
- new net: C?.2, R?.1, R?.1, U?.5 (+)
- new net: C?.2, R?.1, R?.1, U?.10 (+)
- new net: C?.2, R?.1, R?.2, U?.8
- new net: C?.1, R?.1, R?.2, U?.9 (-)
- new net: R?.1, R?.2, SW?.2
- new net: D?.2 (A), R?.1
- new net BOOT0_{SW}: R?.1, SW?.2 (B)
- new net BOOT_{0}: R?.2, U?.1 (BOOT0)
- new net OSC_{MCOUT}: R?.2, U?.3 (PF1)
- new net SENSE_{U}: R?.1, U?.6 (PA0)
- new net SENSE_{V}: R?.1, U?.7 (PA1)
- new net SENSE_{W}: R?.1, U?.8 (PA2)
- new net SPEED/ANGLE: U?.9 (PA3)
- new net ~{USER_{INPUT}}: C?.1, R?.1, U?.10 (PA4)
- no-connect marks 3 -> 11
Other:
- note added: "Push-pull signal"
- note removed: "+3V3 = 1.27*(1+806/500) = 3.31724V"
- moved on the sheet: C1, C11, C12, C18, C19, C2, C21, C24, C3, C4, D1, D2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
