File: BLDC_driver_small.kicad_sch (KiCad schematic)
At the start: 70 parts, among them J1 1x02 Terminal, J2 1x03 Terminal, J3 Conn_02x05_Odd_Even, J4 Conn_01x04, Q1 Q_PMOS_GDS, SW1 RST_SW, SW2 SW_SPDT, SW3 SW_Push_45deg, U1 STM32F030F4Px, U2 L6230Q, U3 TLS850C2TEV33, U4 TSV994, Y1 48MHz

Commit message: 150323
Parts:
- added R26, R27: 4k7, Resistor_SMD:R_0402_1005Metric, symbol Device:R_Small
- RV1: footprint Potentiometer_SMD:Potentiometer_Vishay_TS53YL_Vertical -> Potentiometer_SMD:Potentiometer_Bourns_3314S_Horizontal
Connections:
- net +3V3: now also R26.1, R27.1
- net I2C_{SCL}: now also R26.2
- net I2C_{SDA}: now also R27.2
- net OP3+: now also U4.12 (+); no longer U4.10 (+)
- net OP3-: now also U4.13 (-); no longer U4.9 (-)
- net OP3_{O}: now also U4.14; no longer U4.8
Changed lines of the file:
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@@
     (stroke (width 0) (type default) (color 0 0 0 0))
   )
+  (wire (pts (xy 255.27 78.74) (xy 255.27 80.01))
+    (stroke (width 0) (type default) (color 0 0 0 0))
+  )
   (wire (pts (xy 127 158.75) (xy 127 154.94))
     (stroke (width 0) (type default) (color 0 0 0 0))
@@
     (stroke (width 0) (type default) (color 0 0 0 0))
   )
+  (wire (pts (xy 248.92 85.09) (xy 248.92 87.63))
+    (stroke (width 0) (type default) (color 0 0 0 0))
+  )
   (wire (pts (xy 91.44 99.06) (xy 91.44 101.6))
     (stroke (width 0) (type default) (color 0 0 0 0))
@@
     (stroke (width 0) (type default) (color 0 0 0 0))
   )
+  (wire (pts (xy 248.92 78.74) (xy 248.92 80.01))
+    (stroke (width 0) (type default) (color 0 0 0 0))
+  )
   (wire (pts (xy 69.85 39.37) (xy 68.58 39.37))
     (stroke (width 0) (type default) (color 0 0 0 0))
@@
     (stroke (width 0) (type default) (color 0 0 0 0))
   )
+  (wire (pts (xy 255.27 85.09) (xy 255.27 87.63))
+    (stroke (width 0) (type default) (color 0 0 0 0))
+  )
   (wire (pts (xy 254 49.53) (xy 261.62 49.53))
     (stroke (width 0) (type default) (color 0 0 0 0))
@@
     (effects (font (size 1 1)) (justify right bottom))
   )
+  (label "I2C_{SDA}" (at 255.27 87.63 0)
+    (effects (font (size 1 1)) (justify left bottom))
+  )
   (label "BOOT_{0}" (at 201.93 92.71 180)
     (effects (font (size 1 1)) (justify right bottom))
@@
     (effects (font (size 1 1)) (justify left bottom))
   )
+  (label "I2C_{SCL}" (at 248.92 87.63 0)
+    (effects (font (size 1 1)) (justify left bottom))
+  )
   (label "SENSE_{V}-" (at 83.82 106.68 270)
     (effects (font (size 1 1)) (justify right bottom))
@@
     (effects (font (size 1 1)) (justify left bottom))
   )
+  (symbol (lib_id "power:+3V3") (at 248.92 78.74 0) (unit 1)
+    (in_bom yes) (on_board yes)
+    (property "Reference" "#PWR014" (id 0) (at 248.92 82.55 0)
+      (effects (font (size 1.27 1.27)) hide)
+    )
+    (property "Value" "+3V3" (id 1) (at 245.11 77.47 0)
+      (effects (font (size 1 1)))
+    )
+    (property "Footprint" "" (id 2) (at 248.92 78.74 0)
+      (effects (font (size 1.27 1.27)) hide)
+    )
+    (property "Datasheet" "" (id 3) (at 248.92 78.74 0)
+      (effects (font (size 1.27 1.27)) hide)
+    )
+    (pin "1")
+  )
   (symbol (lib_id "power:+3.3VA") (at 219.71 81.28 0) (unit 1)
     (in_bom yes) (on_board yes)
@@
     (pin "2")
   )
+  (symbol (lib_id "Device:R_Small") (at 255.27 82.55 0) (unit 1)
+    (in_bom yes) (on_board yes)
+    (property "Reference" "R27" (id 0) (at 257.81 82.55 90)
+      (effects (font (size 1 1)))
+    )
+    (property "Value" "4k7" (id 1) (at 255.27 82.55 90)
+      (effects (font (size 1 1)))
+    )
+    (property "Footprint" "Resistor_SMD:R_0402_1005Metric" (id 2) (at 255.27 82.55 0)
+      (effects (font (size 1.27 1.27)) hide)
+    )
+    (property "Datasheet" "~" (id 3) (at 255.27 82.55 0)
+      (effects (font (size 1.27 1.27)) hide)
+    )
+    (pin "1")
+    (pin "2")
+  )
   (symbol (lib_id "fraciscoestar:TLS850C2TEV33") (at 76.2 24.13 0) (unit 1)
     (in_bom yes) (on_board yes) (fields_autoplaced)
@@
     (pin "4")
   )
+  (symbol (lib_id "Device:R_Small") (at 248.92 82.55 0) (unit 1)
+    (in_bom yes) (on_board yes)
+    (property "Reference" "R26" (id 0) (at 251.46 82.55 90)
+      (effects (font (size 1 1)))
+    )
+    (property "Value" "4k7" (id 1) (at 248.92 82.55 90)
+      (effects (font (size 1 1)))
+    )
+    (property "Footprint" "Resistor_SMD:R_0402_1005Metric" (id 2) (at 248.92 82.55 0)
+      (effects (font (size 1.27 1.27)) hide)
+    )
+    (property "Datasheet" "~" (id 3) (at 248.92 82.55 0)
+      (effects (font (size 1.27 1.27)) hide)
+    )
+    (pin "1")
+    (pin "2")
+  )
   (symbol (lib_id "Device:Crystal_GND24_Small") (at 162.56 91.44 0) (mirror y) (unit 1)
     (in_bom yes) (on_board yes)
@@
     (pin "1")
   )
-  (symbol (lib_id "Amplifier_Operational:TSV994") (at 256.54 147.32 0) (unit 3)
+  (symbol (lib_id "Amplifier_Operational:TSV994") (at 256.54 147.32 0) (unit 4)
     (in_bom yes) (on_board yes) (fields_autoplaced)
     (property "Reference" "U4" (id 0) (at 256.54 137.16 0))
@@
       (effects (font (size 1 1)) (justify right))
     )
-    (property "Footprint" "Potentiometer_SMD:Potentiometer_Vishay_TS53YL_Vertical" (id 2) (at 175.26 66.04 0)
+    (property "Footprint" "Potentiometer_SMD:Potentiometer_Bourns_3314S_Horizontal" (id 2) (at 175.26 66.04 0)
       (effects (font (size 1.27 1.27)) hide)
     )
@@
     (pin "2")
   )
-  (symbol (lib_id "Amplifier_Operational:TSV994") (at 121.92 181.61 0) (unit 4)
+  (symbol (lib_id "Amplifier_Operational:TSV994") (at 121.92 181.61 0) (unit 3)
     (in_bom yes) (on_board yes) (fields_autoplaced)
     (property "Reference" "U4" (id 0) (at 121.92 171.45 0))
@@
     (pin "4")
   )
+  (symbol (lib_id "power:+3V3") (at 255.27 78.74 0) (unit 1)
+    (in_bom yes) (on_board yes)
+    (property "Reference" "#PWR022" (id 0) (at 255.27 82.55 0)
+      (effects (font (size 1.27 1.27)) hide)
+    )
+    (property "Value" "+3V3" (id 1) (at 251.46 77.47 0)
+      (effects (font (size 1 1)))
+    )
+    (property "Footprint" "" (id 2) (at 255.27 78.74 0)
+      (effects (font (size 1.27 1.27)) hide)
+    )
+    (property "Datasheet" "" (id 3) (at 255.27 78.74 0)
+      (effects (font (size 1.27 1.27)) hide)
+    )
+    (pin "1")
+  )
   (symbol (lib_id "Device:LED") (at 80.01 39.37 180) (unit 1)
     (in_bom yes) (on_board yes)
@@
       (reference "#PWR013") (unit 1) (value "+24V") (footprint "")
     )
+    (path "/00ecbc50-5b22-4ea0-8efc-ce296f565c3c"
+      (reference "#PWR014") (unit 1) (value "+3V3") (footprint "")
+    )
     (path "/c7060751-3670-4ece-80eb-6d4896f7e327"
       (reference "#PWR015") (unit 1) (value "GND") (footprint "")
@@
       (reference "#PWR021") (unit 1) (value "GND") (footprint "")
     )
+    (path "/bf085de1-006c-4118-ae43-14fac7111789"
+      (reference "#PWR022") (unit 1) (value "+3V3") (footprint "")
+    )
     (path "/2cd105ed-2668-4ecd-bc8f-24ca91d0be69"
       (reference "#PWR023") (unit 1) (value "+24V") (footprint "")
@@
       (reference "R25") (unit 1) (value "0R") (footprint "Resistor_SMD:R_0402_1005Metric")
     )
+    (path "/14103578-0fd1-4027-8e21-143fbb9a860b"
+      (reference "R26") (unit 1) (value "4k7") (footprint "Resistor_SMD:R_0402_1005Metric")
+    )
+    (path "/114b8cd9-f65e-4437-8cef-2c97c70dd207"
+      (reference "R27") (unit 1) (value "4k7") (footprint "Resistor_SMD:R_0402_1005Metric")
+    )
     (path "/68ae5740-82b8-4a31-9367-e9051566070d"
-      (reference "RV1") (unit 1) (value "R_Potentiometer") (footprint "Potentiometer_SMD:Potentiometer_Vishay_TS53YL_Vertical")
+      (reference "RV1") (unit 1) (value "R_Potentiometer") (footprint "Potentiometer_SMD:Potentiometer_Bourns_3314S_Horizontal")
     )
     (path "/ab471b0c-d944-4c51-82e9-447cab6ec909"
@@
       (reference "U4") (unit 2) (value "TSV994") (footprint "Package_SO:TSSOP-14_4.4x5mm_P0.65mm")
     )
-    (path "/5d2b2bdd-bc8b-445e-993c-13779711a90c"
+    (path "/beef8626-8783-4d5b-a7c5-28cdc51c71c3"
       (reference "U4") (unit 3) (value "TSV994") (footprint "Package_SO:TSSOP-14_4.4x5mm_P0.65mm")
     )
-    (path "/beef8626-8783-4d5b-a7c5-28cdc51c71c3"
+    (path "/5d2b2bdd-bc8b-445e-993c-13779711a90c"
       (reference "U4") (unit 4) (value "TSV994") (footprint "Package_SO:TSSOP-14_4.4x5mm_P0.65mm")
     )

Commit message: 160323
Parts:
- added C8: 100n, Capacitor_SMD:C_0402_1005Metric, symbol Device:C_Small
- added H1, H2, H3: MountingHole, MountingHole:MountingHole_2.2mm_M2, symbol Mechanical:MountingHole
- C7: value 220n -> 100n
Connections:
- net +24V: now also C8.1
- net +3V3: now also D4.2 (A); no longer R2.2
- net GND: now also R2.1, C8.2; no longer D4.1 (K)
- net OP3+: now also U4.10 (+); no longer U4.12 (+)
- net OP3-: now also U4.9 (-); no longer U4.13 (-)
- net OP3_{O}: now also U4.8; no longer U4.14
- new net: D4.1 (K), R2.2
Other:
- moved on the sheet: D4, R2

Commit message: 160323-2
Parts:
- F1: footprint Resistor_SMD:R_0805_2012Metric -> Fuse:Fuse_1206_3216Metric
Connections:
- net ENABLE: now also U1.9 (PA3); no longer U1.11 (PA5)
- net GND: no longer C1.2, C13.2, C19.2, C20.2, C21.1, C23.1, C25.1, C4.2, C5.2, C6.2, C7.2, C8.2, J1.2 (Pin_2), R1.1, R12.2, R17.2, R22.2, R3.2, R4.2, R5.2, U2.1 (GND), U2.2 (NC), U2.21 (GND), U2.3 (NC), U2.4 (NC), U2.5 (NC), U2.6 (NC), U2.7 (NC), U2.8 (NC), U4.11 (V-)
- net PWM_{U}: now also U1.12 (PA6); no longer U1.14 (PB1)
- net PWM_{V}: now also U1.14 (PB1); no longer U1.12 (PA6)
- net SENSE_{U}: now also R20.1; no longer R15.1
- net SENSE_{U}+: now also R16.2; no longer R11.2
- net SENSE_{V}: now also R15.1; no longer R20.1
- net SENSE_{V}+: now also R11.2; no longer R16.2
- net SPEED/ANGLE: now also U1.10 (PA4); no longer U1.9 (PA3)
- net ~{USER_{INPUT}}: now also U1.11 (PA5); no longer U1.10 (PA4)
- net V_{pwr}: now reaches F1.1, J1.1 (Pin_1)
- net V_{pwrfuse}: now reaches F1.2, Q1.2 (D)
- new net GNDA: C13.2, C19.2, C20.2, C21.1, C23.1, C25.1, C4.2, C5.2, C6.2, U4.11 (V-)
- new net GNDPWR: C1.2, C7.2, C8.2, J1.2 (Pin_2), R1.1, R12.2, R17.2, R22.2, R3.2, R4.2, R5.2, U2.1 (GND), U2.2 (NC), U2.21 (GND), U2.3 (NC), U2.4 (NC), U2.5 (NC), U2.6 (NC), U2.7 (NC), U2.8 (NC)

Commit message: 170323-v1.0
Parts:
- SW3: footprint Button_Switch_SMD:SW_SPST_B3U-1000P -> Button_Switch_SMD:SW_SPST_B3S-1000
Connections:
- net GND: no longer C2.2
- net GNDPWR: now also C2.2
Changed lines of the file:
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@@
   (junction (at 110.49 21.59) (diameter 0) (color 0 0 0 0)
   )
-  (junction (at 73.66 33.02) (diameter 0) (color 0 0 0 0)
-  )
   (junction (at 76.2 121.92) (diameter 0) (color 0 0 0 0)
   )
@@
     (stroke (width 0) (type default) (color 0 0 0 0))
   )
-  (wire (pts (xy 64.77 27.94) (xy 64.77 33.02))
+  (wire (pts (xy 64.77 27.94) (xy 64.77 35.56))
     (stroke (width 0) (type default) (color 0 0 0 0))
   )
@@
     (stroke (width 0) (type default) (color 0 0 0 0))
   )
-  (wire (pts (xy 64.77 33.02) (xy 73.66 33.02))
-    (stroke (width 0) (type default) (color 0 0 0 0))
-  )
   (wire (pts (xy 118.11 137.16) (xy 118.11 135.89))
     (stroke (width 0) (type default) (color 0 0 0 0))
@@
       (effects (font (size 1 1)) (justify right))
     )
-    (property "Footprint" "Button_Switch_SMD:SW_SPST_B3U-1000P" (id 2) (at 256.54 44.45 0)
+    (property "Footprint" "Button_Switch_SMD:SW_SPST_B3S-1000" (id 2) (at 256.54 44.45 0)
       (effects (font (size 1.27 1.27)) hide)
     )
@@
     (pin "2")
   )
+  (symbol (lib_id "power:GNDPWR") (at 64.77 35.56 0) (unit 1)
+    (in_bom yes) (on_board yes)
+    (property "Reference" "#PWR0107" (id 0) (at 64.77 40.64 0)
+      (effects (font (size 1.27 1.27)) hide)
+    )
+    (property "Value" "GNDPWR" (id 1) (at 64.77 39.37 0)
+      (effects (font (size 1 1)))
+    )
+    (property "Footprint" "" (id 2) (at 64.77 36.83 0)
+      (effects (font (size 1.27 1.27)) hide)
+    )
+    (property "Datasheet" "" (id 3) (at 64.77 36.83 0)
+      (effects (font (size 1.27 1.27)) hide)
+    )
+    (pin "1")
+  )
   (symbol (lib_id "Connector_Generic:Conn_02x05_Odd_Even") (at 215.9 43.18 0) (unit 1)
     (in_bom yes) (on_board yes) (fields_autoplaced)
@@
       (reference "#PWR0106") (unit 1) (value "GNDPWR") (footprint "")
     )
+    (path "/adcfbdd3-df72-4e9c-a107-14605a37a9cc"
+      (reference "#PWR0107") (unit 1) (value "GNDPWR") (footprint "")
+    )
     (path "/714bd957-ff2f-42b8-93c8-afb91a19a249"
       (reference "C1") (unit 1) (value "100u") (footprint "Capacitor_SMD:CP_Elec_10x12.5")
@@
     )
     (path "/95455416-00c5-4ded-83a7-e6055f50ab9b"
-      (reference "SW3") (unit 1) (value "SW_Push_45deg") (footprint "Button_Switch_SMD:SW_SPST_B3U-1000P")
+      (reference "SW3") (unit 1) (value "SW_Push_45deg") (footprint "Button_Switch_SMD:SW_SPST_B3S-1000")
     )
     (path "/669b5855-e147-4d37-8788-ac68cca09c3d"

Commit message: v190323-2
Parts:
- added NT1, NT2: NetTie_2, NetTie:NetTie-2_SMD_Pad2.0mm, symbol Device:NetTie_2
- added NT3: NetTie_2, NetTie:NetTie-2_THT_Pad0.3mm, symbol Device:NetTie_2
- added NT4, NT5, NT6: NetTie_2, NetTie:NetTie-2_SMD_Pad0.5mm, symbol Device:NetTie_2
Connections:
- net GND: now also NT2.2, NT3.1
- net GNDA: now also NT3.2
- net GNDPWR: now also NT1.2, NT4.1, NT5.1, NT6.1; no longer J1.2 (Pin_2), R1.1, R12.2, R17.2, R22.2
- new net GNDREF: J1.2 (Pin_2), NT1.1, NT2.1, R1.1
- new net SENSE_{U}-: NT4.2, R17.2
- new net SENSE_{V}-: NT5.2, R12.2
- new net SENSE_{W}-: NT6.2, R22.2

Commit message: 200323-final
Parts:
- added NT7, NT8, NT9: NetTie_2, NetTie:NetTie-2_SMD_Pad0.5mm, symbol Device:NetTie_2
- NT3: footprint NetTie:NetTie-2_THT_Pad0.3mm -> NetTie:NetTie-2_SMD_Pad0.5mm
Connections:
- net GND: now also NT7.1, NT8.1, NT9.1
- net GNDA: now also NT7.2, NT8.2, NT9.2
Other:
- moved on the sheet: NT2

Commit message: v1.0
Parts:
- removed F1: Polyfuse, Fuse:Fuse_1206_3216Metric, symbol Device:Polyfuse_Small
- C1: footprint Capacitor_SMD:CP_Elec_10x12.5 -> Capacitor_SMD:CP_Elec_10x10.5; MPN (none) -> 865060757007
- C10: MPN (none) -> TMK105B7224KV-FR
- C11, C19: MPN (none) -> GRM155C61E475ME15J
- C12, C13, C14, C15, C20, C7, C8: MPN (none) -> 885012205092
- C16: MPN (none) -> GRM155R71E562JA01D
- C17, C18: value TBD -> 30p; MPN (none) -> 04025A300FAT2A
- C2: MPN (none) -> UMK107BJ105KA-T
- C21, C23, C25: MPN (none) -> MAASH105SB7681KFCA01
- C22, C24, C26: MPN (none) -> C0402C101K3RACAUTO
- C3: MPN (none) -> GRM188R6YA475KE15J
- C4, C5: MPN (none) -> EMK105BJ105KV8F
- C6, C9: MPN (none) -> UMK105B7103KV-F
- D1: MPN (none) -> MMSZ5252C-G3-08
- D2, D3: MPN (none) -> 1N4148X-TP
- D4: MPN (none) -> 150060GS75000
- J1: MPN (none) -> 1711026
- J2: MPN (none) -> 1711039
- J3: MPN (none) -> 5103310-1
- J4: MPN (none) -> 90147-1204
- L1: MPN (none) -> LQG18HN39NJ00D
- Q1: MPN (none) -> SQ2319ADS-T1_BE3
- R1, R6, R9: MPN (none) -> ERJ-2RKF1002X
- R10, R12, R13, R14, R17, R18, R19, R2, R22, R23, R24: MPN (none) -> ERJ-2RKF2201X
- R11, R16, R21: MPN (none) -> ERJ-2RKF6800X
- R15, R20, R25: MPN (none) -> ERJ-2GE0R00X
- R26, R27: MPN (none) -> ERJ-2RKF4701X
- R3, R4, R5: MPN (none) -> RCWE1210R330FKEA
- R7: MPN (none) -> ERJ-2RKF47R0X
- R8: MPN (none) -> ERJ-2RKF1003X
- RV1: MPN (none) -> 3314J-1-204E
- SW1, SW3: MPN (none) -> K2-1157SP-B3SW-01
- SW2: MPN (none) -> SK-3296S-01-L1
- U1: MPN (none) -> STM32F030F4P6
- U2: MPN (none) -> L6230Q
- U3: MPN (none) -> TLS850C2TEV33
- U4: MPN (none) -> TSV994
- Y1: MPN (none) -> 7B048000R01
Connections:
- net V_{pwrfuse} is gone; now on net V_{pwr}: Q1.2 (D)
