File: BLDC_driver_small.kicad_pcb (KiCad board)
At the start: 2 copper layers, 50 x 50 mm, 54 parts, among them J1 1x02 Terminal, J2 1x03 Terminal, Q1 Q_PMOS_GDS, SW1 RST_SW, SW2 SW_SPDT, U1 NCP786L, U2 L6230PD, U3 ADS131M03IPWR, U4 STM32F030K6Tx, Y1 16MHz

Commit message: 130323
Parts:
- added F1: Polyfuse, Resistor_SMD:R_0805_2012Metric, F.Cu at (115.4, 63.5)
- C23: footprint Capacitor_SMD:C_0603_1608Metric -> Resistor_SMD:R_0402_1005Metric
- R10, R12, R13, R15, R4, R8: value 1M -> 500k; footprint Resistor_SMD:R_0603_1608Metric -> Resistor_SMD:R_0402_1005Metric
- R11: footprint Resistor_SMD:R_0603_1608Metric -> Resistor_SMD:R_0402_1005Metric
- moved C20 134.8 mm to (164.0, 102.2), turned to -90 degrees
- moved C23 121.4 mm to (174.0, 98.3), turned to 90 degrees
- moved R8 117.8 mm to (162.4, 98.8)
- moved R13 116.5 mm to (162.4, 101.9)
- moved R4 116.0 mm to (162.4, 97.8)
- moved R15 115.7 mm to (162.4, 102.9)
- moved R12 115.4 mm to (162.4, 99.8)
- moved R10 115.3 mm to (162.4, 100.8)
- moved C17 114.8 mm to (164.0, 100.4), turned to 90 degrees
- moved C16 111.1 mm to (164.0, 98.3), turned to -90 degrees
- moved D1 86.9 mm to (119.4, 59.4), turned to 180 degrees
- moved R11 82.2 mm to (134.9, 84.1), turned to -90 degrees
- moved Q1 76.3 mm to (119.4, 62.7)
- moved L1 75.3 mm to (126.0, 59.4)
- moved C19 60.2 mm to (101.2, 44.3), turned to 90 degrees
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Routing:
- net GND: track 0.00 -> 8.27 mm
- net +24V: track 0.00 -> 4.12 mm
- net +3V3: track 0.00 -> 2.91 mm
- net +3.3VA: track 0.00 -> 1.84 mm

Commit message: 130323-2
Parts:
- C4: footprint Capacitor_SMD:CP_Elec_6.3x5.4 -> Capacitor_SMD:CP_Elec_10x12.5
- R5, R7, R9: value 10m -> 0.33
- U2: value L6230PD -> L6230Q; footprint fraciscoestar:PowerSO36 -> fraciscoestar:VFQFPN32
- moved U2 4.57 mm to (112.6, 104.4)
- moved C4 2.93 mm to (113.3, 77.4)
Connections:
- U2 pad 10: /ENA_{U} -> unconnected-(U2-Pad10)
- U2 pad 11: /PWM_{W} -> unconnected-(U2-Pad11)
- U2 pad 12: /SENSE_{U}+ -> /SENSE_{W}+
- U2 pad 13: unconnected-(U2-Pad13) -> /PWM_{V}
- U2 pad 14: unconnected-(U2-Pad14) -> /ENA_{V}
- U2 pad 15: /OUT_{U} -> unconnected-(U2-Pad15)
- U2 pad 16: unconnected-(U2-Pad16) -> /ENA_{W}
- U2 pad 17: unconnected-(U2-Pad17) -> /V_{BOOT}
- U2 pad 18: GND -> unconnected-(U2-Pad18)
- U2 pad 19: GND -> /OUT_{W}
- U2 pad 20: unconnected-(U2-Pad20) -> +24V
- U2 pad 21: unconnected-(U2-Pad21) -> GND
- U2 pad 22: /ENA_{DRV} -> +24V
- U2 pad 23: unconnected-(U2-Pad23) -> /OUT_{V}
- U2 pad 24: unconnected-(U2-Pad24) -> Net-(C21-Pad2)
- U2 pad 25: /SENSE_{W}+ -> /SENSE_{V}+
- U2 pad 26: /PWM_{V} -> /PWM_{U}
- U2 pad 27: /ENA_{V} -> /ENA_{U}
- U2 pad 28: unconnected-(U2-Pad28) -> /PWM_{W}
- U2 pad 29: /ENA_{W} -> /SENSE_{U}+
- U2 pad 30: /V_{BOOT} -> unconnected-(U2-Pad30)
- U2 pad 31: unconnected-(U2-Pad31) -> /OUT_{U}
- U2 pad 32: /OUT_{W} -> unconnected-(U2-Pad32)
- U2 pad 4: +24V -> unconnected-(U2-Pad4)
- U2 pad 5: /OUT_{V} -> unconnected-(U2-Pad5)
- U2 pad 7: Net-(C21-Pad2) -> unconnected-(U2-Pad7)
- U2 pad 8: /SENSE_{V}+ -> unconnected-(U2-Pad8)
- U2 pad 9: /PWM_{U} -> /ENA_{DRV}
Routing:
- net GND: track 8.27 -> 4.70 mm
- net +24V: track 4.12 -> 0.59 mm

Commit message: 140323
Parts:
- removed C8: 100n, Capacitor_SMD:C_0402_1005Metric
- removed L2: 39n, Inductor_SMD:L_0603_1608Metric
- added C25: 680p, Capacitor_SMD:C_0402_1005Metric, F.Cu at (251.9, 84.7)
- added C26: 100p, Capacitor_SMD:C_0402_1005Metric, F.Cu at (260.8, 87.1)
- added D4: LED, LED_SMD:LED_0603_1608Metric, F.Cu at (169.5, 55.0)
- added J3: Conn_02x05_Odd_Even, Connector_PinHeader_2.54mm:PinHeader_2x05_P2.54mm_Vertical, F.Cu at (147.1, 90.9)
- added J4: Conn_01x04, Connector_PinHeader_2.54mm:PinHeader_1x04_P2.54mm_Vertical, F.Cu at (147.1, 102.2)
- added R16: 680, Resistor_SMD:R_0402_1005Metric, F.Cu at (244.9, 105.4)
- added R17: 2k2, Resistor_SMD:R_0402_1005Metric, F.Cu at (247.2, 106.5)
- added R18: 2k2, Resistor_SMD:R_0402_1005Metric, F.Cu at (247.6, 104.9)
- added R19: 2k2, Resistor_SMD:R_0402_1005Metric, F.Cu at (248.2, 108.7)
- added R20: 0R, Resistor_SMD:R_0402_1005Metric, F.Cu at (250.2, 109.2)
- added R21: 680, Resistor_SMD:R_0402_1005Metric, F.Cu at (250.3, 85.1)
- added R22: 2k2, Resistor_SMD:R_0402_1005Metric, F.Cu at (250.3, 86.3)
- added R23: 2k2, Resistor_SMD:R_0402_1005Metric, F.Cu at (253.1, 84.7)
- added R24: 2k2, Resistor_SMD:R_0402_1005Metric, F.Cu at (260.8, 86.0)
- added R25: 0R, Resistor_SMD:R_0402_1005Metric, F.Cu at (268.2, 85.2)
- added RV1: R_Potentiometer, Potentiometer_SMD:Potentiometer_Vishay_TS53YL_Vertical, F.Cu at (108.0, 22.6)
- added SW3: SW_Push_45deg, Button_Switch_SMD:SW_SPST_B3U-1000P, F.Cu at (67.1, 58.0)
- C1: value 1u -> 100u; footprint Capacitor_SMD:C_0603_1608Metric -> Capacitor_SMD:CP_Elec_10x12.5
- C10: value 100n -> 220n
- C11: value 100n -> 4u7; footprint Capacitor_SMD:C_0603_1608Metric -> Capacitor_SMD:C_0402_1005Metric
- C12: footprint Capacitor_SMD:C_0603_1608Metric -> Capacitor_SMD:C_0402_1005Metric
- C14, C15: value 1u -> 100n
- C16: value 1n -> 5n6
- C17: value 1n -> TBD
- C19: value TBD -> 4u7
- C20: value 1n -> 100n
- C21: value 10n -> 680p; footprint Capacitor_SMD:C_0603_1608Metric -> Capacitor_SMD:C_0402_1005Metric
- C22: value 5n6 -> 100p
- C23: value 220n -> 680p; footprint Resistor_SMD:R_0402_1005Metric -> Capacitor_SMD:C_0402_1005Metric
- C24: value 220n -> 100p; footprint Capacitor_SMD:C_0603_1608Metric -> Capacitor_SMD:C_0402_1005Metric
- C3: value 10n -> 4u7
- C4: value 100u -> 1u; footprint Capacitor_SMD:CP_Elec_10x12.5 -> Capacitor_SMD:C_0402_1005Metric
- C5: value 2u2 -> 1u; footprint Capacitor_SMD:C_0805_2012Metric -> Capacitor_SMD:C_0402_1005Metric
- C6: value 4u7 -> 10n; footprint Capacitor_SMD:C_0603_1608Metric -> Capacitor_SMD:C_0402_1005Metric
- C7: value 4u7 -> 220n; footprint Capacitor_SMD:C_0603_1608Metric -> Capacitor_SMD:C_0402_1005Metric
- C9: value 100n -> 10n
- D2, D3: footprint Diode_SMD:D_SOD-323 -> Diode_SMD:D_SOD-523
- L1: value 10u -> 39n; footprint Inductor_SMD:L_6.3x6.3_H3 -> Inductor_SMD:L_0603_1608Metric
- R1: value 806k -> 10k; footprint Resistor_SMD:R_0603_1608Metric -> Resistor_SMD:R_0402_1005Metric
- R10, R12, R13: value 500k -> 2k2
- R11: value 47R -> 680
- R14: value 100k -> 2k2; footprint Resistor_SMD:R_0603_1608Metric -> Resistor_SMD:R_0402_1005Metric
- R15: value 500k -> 0R
- R2: value 10k -> 2k2; footprint Resistor_SMD:R_0603_1608Metric -> Resistor_SMD:R_0402_1005Metric
- R3: value 500k -> 0.33; footprint Resistor_SMD:R_0603_1608Metric -> Resistor_SMD:R_1210_3225Metric
- R4: value 500k -> 0.33; footprint Resistor_SMD:R_0402_1005Metric -> Resistor_SMD:R_1210_3225Metric
- R6: footprint Resistor_SMD:R_0603_1608Metric -> Resistor_SMD:R_0402_1005Metric
- R7: value 0.33 -> 47R; footprint Resistor_SMD:R_1210_3225Metric -> Resistor_SMD:R_0402_1005Metric
- R8: value 500k -> 100k
- R9: value 0.33 -> 10k; footprint Resistor_SMD:R_1210_3225Metric -> Resistor_SMD:R_0402_1005Metric
- U1: value NCP786L -> STM32F030F4Px; footprint Package_TO_SOT_SMD:SOT-223 -> Package_SO:TSSOP-20_4.4x6.5mm_P0.65mm
- U3: value ADS131M03IPWR -> TLS850C2TEV33; footprint Package_SO:TSSOP-20_4.4x6.5mm_P0.65mm -> fraciscoestar:PG-TO252-5
- U4: value STM32F030K6Tx -> TSV994; footprint Package_QFP:LQFP-32_7x7mm_P0.8mm -> Package_SO:TSSOP-14_4.4x5mm_P0.65mm
- Y1: value 16MHz -> 48MHz
- moved C22 210.1 mm to (248.2, 99.1)
- moved R14 204.1 mm to (248.2, 100.2), turned to 180 degrees
- moved C19 143.0 mm to (231.9, 102.3), turned to 0 degrees
- moved C24 136.1 mm to (248.2, 107.6), turned to 0 degrees
- moved C21 131.8 mm to (246.5, 102.9)
- moved U4 120.3 mm to (253.3, 103.9), turned to 0 degrees
- moved C13 118.4 mm to (133.9, 112.1), turned to 180 degrees
- moved R11 111.5 mm to (244.9, 102.4), turned to 180 degrees
- moved C14 102.0 mm to (71.4, 60.1)
- moved R6 101.2 mm to (133.9, 109.5)
- moved C15 100.9 mm to (90.2, 36.5), turned to 0 degrees
- moved J2 91.6 mm to (62.8, 26.4), turned to 0 degrees
- moved R15 87.9 mm to (250.2, 98.6), turned to -90 degrees
- moved R10 85.8 mm to (114.1, 29.9)
- moved R13 85.2 mm to (247.6, 102.9), turned to -90 degrees
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Connections:
- net Net-(R6-Pad1) renamed /BOOT0_{SW}
- C1 pad 1: +3V3 -> +24V
- C10 pad 1: +3.3VA -> +24V
- C10 pad 2: GND -> /V_{BOOT}
- C11 pad 1: +24V -> +3V3
- C12 pad 1: +24V -> +3V3
- C13 pad 1: /NRST -> +3.3VA
- C14 pad 1: +3.3VA -> /NRST
- C15 pad 1: +3V3 -> /~{USER_{INPUT}}
- C16 pad 1: /ADC_{IN0}+ -> /ENA_{DRV}
- C16 pad 2: /ADC_{IN0}- -> GND
- C17 pad 1: /ADC_{IN1}+ -> /OSC_{OUT}
- C17 pad 2: /ADC_{IN1}- -> GND
- C18 pad 1: /OSC_{OUT} -> /OSC_{IN}
- C19 pad 1: /OSC_{IN} -> +3.3VA
- C2 pad 1: +3.3VA -> +24V
- C20 pad 1: /ADC_{IN2}+ -> +3.3VA
- C20 pad 2: /ADC_{IN2}- -> GND
- C21 pad 1: Net-(C21-Pad1) -> GND
- C21 pad 2: Net-(C21-Pad2) -> /OP1+
- C22 pad 1: /ENA_{DRV} -> /OP1-
- C22 pad 2: GND -> /OP1_{O}
- C23 pad 1: +1V2 -> GND
- C23 pad 2: GND -> /OP2+
- C24 pad 1: +24V -> /OP2-
- C24 pad 2: /V_{BOOT} -> /OP2_{O}
- C3 pad 1: +3.3VA -> +3V3
- C4 pad 1: +24V -> +3V3
- C5 pad 1: +24V -> +3.3VA
- C6 pad 1: +3V3 -> +3.3VA
- C7 pad 1: +3V3 -> +24V
- C9 pad 1: +3V3 -> Net-(C9-Pad1)
- C9 pad 2: GND -> /V_{CP}
- D1 pad 1: Net-(D1-Pad1) -> +24V
- D2 pad 1: Net-(C21-Pad1) -> Net-(C9-Pad1)
- D3 pad 2: Net-(C21-Pad1) -> Net-(C9-Pad1)
- L1 pad 1: Net-(D1-Pad1) -> +3V3
- L1 pad 2: +24V -> +3.3VA
- Q1 pad 3: Net-(D1-Pad1) -> +24V
- R1 pad 1: Net-(R1-Pad1) -> GND
- R1 pad 2: +3V3 -> Net-(D1-Pad2)
- R10 pad 1: /SENSE_{V}+ -> /~{USER_{INPUT}}
- R10 pad 2: /ADC_{IN1}+ -> Net-(R10-Pad2)
- R11 pad 1: /OSC_{OUT} -> /OP1+
- R11 pad 2: Net-(R11-Pad2) -> /SENSE_{U}+
- R12 pad 1: GND -> /OP1-
- R12 pad 2: /ADC_{IN1}- -> GND
- R13 pad 1: /SENSE_{W}+ -> /OP1+
- R13 pad 2: /ADC_{IN2}+ -> +3.3VA
- R14 pad 1: /ENA_{DRV} -> /OP1_{O}
- R14 pad 2: Net-(R14-Pad2) -> /OP1-
- R15 pad 1: GND -> /SENSE_{U}
- R15 pad 2: /ADC_{IN2}- -> /OP1_{O}
- R2 pad 1: GND -> Net-(D4-Pad2)
- R2 pad 2: Net-(D1-Pad2) -> +3V3
- R3 pad 1: GND -> /SENSE_{U}+
- R3 pad 2: Net-(R1-Pad1) -> GND
- R4 pad 1: /SENSE_{U}+ -> /SENSE_{V}+
- R4 pad 2: /ADC_{IN0}+ -> GND
- R5 pad 1: /SENSE_{U}+ -> /SENSE_{W}+
- R6 pad 2: Net-(R6-Pad2) -> /BOOT_{0}
- R7 pad 1: /SENSE_{V}+ -> /OSC_{OUT}
- R7 pad 2: GND -> /OSC_{MCOUT}
- R8 pad 1: GND -> /ENA_{DRV}
- R8 pad 2: /ADC_{IN0}- -> /ENABLE
- R9 pad 1: /SENSE_{W}+ -> Net-(R10-Pad2)
- R9 pad 2: GND -> +3V3
- U1 pad 1: +24V -> /BOOT_{0}
- U1 pad 2: Net-(R1-Pad1) -> /OSC_{IN}
- U1 pad 3: +3V3 -> /OSC_{MCOUT}
- U1 pad 4: GND -> /NRST
- U2 pad 14: /ENA_{V} -> /ENABLE
- U2 pad 16: /ENA_{W} -> /ENABLE
- U2 pad 2: unconnected-(U2-Pad2) -> GND
- U2 pad 24: Net-(C21-Pad2) -> /V_{CP}
- U2 pad 27: /ENA_{U} -> /ENABLE
- U2 pad 3: unconnected-(U2-Pad3) -> GND
- U2 pad 4: unconnected-(U2-Pad4) -> GND
- U2 pad 5: unconnected-(U2-Pad5) -> GND
- U2 pad 6: unconnected-(U2-Pad6) -> GND
- U2 pad 7: unconnected-(U2-Pad7) -> GND
- U2 pad 8: unconnected-(U2-Pad8) -> GND
- U3 pad 1: +3.3VA -> +24V
- U3 pad 2: GND -> unconnected-(U3-Pad2)
- U3 pad 3: /ADC_{IN0}+ -> GND
- U3 pad 4: /ADC_{IN0}- -> unconnected-(U3-Pad4)
- U3 pad 5: /ADC_{IN1}- -> +3V3
- U4 pad 1: +3V3 -> /OP1_{O}
- U4 pad 10: /~{ADC_{DRDY}} -> /OP3+
- U4 pad 11: /ADC_{SCLK} -> GND
- U4 pad 12: /ADC_{MISO} -> unconnected-(U4-Pad12)
- U4 pad 13: /ADC_{MOSI} -> unconnected-(U4-Pad13)
- U4 pad 14: /~{ADC_{RST}} -> unconnected-(U4-Pad14)
- U4 pad 2: /OSC_{IN} -> /OP1-
- U4 pad 3: Net-(R11-Pad2) -> /OP1+
- U4 pad 4: /NRST -> +3.3VA
- U4 pad 5: +3.3VA -> /OP2+
- U4 pad 6: unconnected-(U4-Pad6) -> /OP2-
- U4 pad 7: unconnected-(U4-Pad7) -> /OP2_{O}
- U4 pad 8: /UART_{TX} -> /OP3_{O}
- U4 pad 9: /UART_{RX} -> /OP3-
Routing:
- net GND: track 4.70 -> 0.00 mm
- net +3V3: track 2.91 -> 0.00 mm
- net +3.3VA: track 1.84 -> 0.00 mm
- net +24V: track 0.59 -> 0.00 mm

Commit message: 150323
Parts:
- added R26: 4k7, Resistor_SMD:R_0402_1005Metric, F.Cu at (143.0, 96.1)
- added R27: 4k7, Resistor_SMD:R_0402_1005Metric, F.Cu at (143.0, 94.1)
- C19, C20: moved to B.Cu
- RV1: footprint Potentiometer_SMD:Potentiometer_Vishay_TS53YL_Vertical -> Potentiometer_SMD:Potentiometer_Bourns_3314S_Horizontal
- moved R25 133.9 mm to (135.8, 105.3), turned to -90 degrees
- moved R24 125.2 mm to (137.3, 106.4), turned to -90 degrees
- moved C26 123.9 mm to (138.4, 106.4), turned to 90 degrees
- moved R19 120.6 mm to (127.7, 114.4)
- moved C21 120.6 mm to (126.0, 108.6)
- moved C23 120.6 mm to (126.0, 110.6)
- moved R11 120.6 mm to (124.4, 108.1)
- moved R13 120.6 mm to (127.1, 108.6)
- moved R15 120.6 mm to (129.7, 104.3)
- moved R16 120.6 mm to (124.4, 111.1)
- moved R18 120.6 mm to (127.1, 110.6)
- moved U4 120.6 mm to (132.8, 109.6)
- moved C22 120.6 mm to (127.7, 104.8)
- moved C24 120.6 mm to (127.7, 113.3)
- moved R12 120.6 mm to (126.7, 107.0)
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Connections:
- U4 pad 10: /OP3+ -> unconnected-(U4-Pad10)
- U4 pad 12: unconnected-(U4-Pad12) -> /OP3+
- U4 pad 13: unconnected-(U4-Pad13) -> /OP3-
- U4 pad 14: unconnected-(U4-Pad14) -> /OP3_{O}
- U4 pad 8: /OP3_{O} -> unconnected-(U4-Pad8)
- U4 pad 9: /OP3- -> unconnected-(U4-Pad9)
Other:
- copper layers 2 -> 6

Commit message: 160323
Parts:
- added C8: 100n, Capacitor_SMD:C_0402_1005Metric, F.Cu at (115.2, 83.0)
- added H1: MountingHole, MountingHole:MountingHole_2.2mm_M2, F.Cu at (146.0, 72.4)
- added H2: MountingHole, MountingHole:MountingHole_2.2mm_M2, F.Cu at (102.0, 72.4)
- added H3: MountingHole, MountingHole:MountingHole_2.2mm_M2, F.Cu at (146.0, 116.4)
- C7: value 220n -> 100n
- moved SW1 87.5 mm to (202.1, 52.2)
- moved SW2 87.5 mm to (211.6, 50.6)
- moved RV1 84.5 mm to (226.8, 134.1)
- moved SW3 84.5 mm to (228.3, 128.8)
- moved R9 84.5 mm to (225.9, 127.6)
- moved J3 78.3 mm to (225.4, 90.7)
- moved J4 78.3 mm to (225.4, 102.0)
- moved D4 71.5 mm to (126.7, 103.4), turned to -90 degrees
- moved R2 71.3 mm to (125.9, 101.3)
- moved C14 70.8 mm to (199.9, 64.6)
- moved C18 70.8 mm to (192.2, 63.6)
- moved R6 70.8 mm to (196.4, 65.1)
- moved C11 70.8 mm to (206.5, 68.9)
- moved C12 70.8 mm to (205.4, 68.9)
- moved C13 70.8 mm to (195.9, 68.4)
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Connections:
- D4 pad 1: GND -> Net-(R2-Pad2)
- D4 pad 2: Net-(D4-Pad2) -> +3V3
- R2 pad 1: Net-(D4-Pad2) -> GND
- R2 pad 2: +3V3 -> Net-(R2-Pad2)
- U4 pad 10: unconnected-(U4-Pad10) -> /OP3+
- U4 pad 12: /OP3+ -> unconnected-(U4-Pad12)
- U4 pad 13: /OP3- -> unconnected-(U4-Pad13)
- U4 pad 14: /OP3_{O} -> unconnected-(U4-Pad14)
- U4 pad 8: unconnected-(U4-Pad8) -> /OP3_{O}
- U4 pad 9: unconnected-(U4-Pad9) -> /OP3-
Routing:
- net /V_{CP}: track 0.00 -> 8.03 mm, vias 0 -> 2
- net /V_{BOOT}: track 0.00 -> 3.14 mm
- net Net-(C9-Pad1): track 0.00 -> 2.86 mm
- net GND: track 0.00 -> 1.68 mm, vias 0 -> 11
- net /OUT_{W}: vias 0 -> 4
- net /OUT_{V}: vias 0 -> 4
- net /OUT_{U}: vias 0 -> 4
- added copper zone on F.Cu, net +24V
- added copper zone on F.Cu, net +3V3
- added copper zone on B.Cu, net /OUT_{U}
- added copper zone on F.Cu, net /OUT_{U}
- added copper zone on B.Cu, net /OUT_{V}
- added copper zone on F.Cu, net /OUT_{V}
- added copper zone on B.Cu, net /OUT_{W}
- added copper zone on F.Cu, net /OUT_{W}
- added copper zone on B.Cu, net GND
- added copper zone on F.Cu, net GND

Commit message: 160323-2
Parts:
- C19, C20: moved to F.Cu
- F1: footprint Resistor_SMD:R_0805_2012Metric -> Fuse:Fuse_1206_3216Metric
- moved J4 85.7 mm to (140.9, 116.8)
- moved SW2 85.7 mm to (128.4, 71.5)
- moved J3 81.0 mm to (147.2, 111.7)
- moved Y1 67.6 mm to (130.0, 93.0)
- moved C11 67.6 mm to (144.4, 95.5)
- moved C12 67.6 mm to (143.3, 95.5)
- moved C13 67.6 mm to (133.8, 95.0)
- moved C17 67.6 mm to (130.0, 95.6)
- moved C18 67.6 mm to (130.0, 90.2)
- moved R26 67.6 mm to (145.8, 94.4)
- moved R27 67.6 mm to (145.8, 92.4)
- moved R6 67.6 mm to (134.3, 91.7)
- moved R7 67.6 mm to (133.8, 93.9)
- moved U1 67.6 mm to (138.8, 95.3)
- moved SW1 67.2 mm to (138.2, 73.1)
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Connections:
- net Net-(F1-Pad1) renamed /V_{pwr}
- net Net-(F1-Pad2) renamed /V_{pwrfuse}
- C1 pad 2: GND -> GNDPWR
- C13 pad 2: GND -> GNDA
- C19 pad 2: GND -> GNDA
- C20 pad 2: GND -> GNDA
- C21 pad 1: GND -> GNDA
- C23 pad 1: GND -> GNDA
- C25 pad 1: GND -> GNDA
- C4 pad 2: GND -> GNDA
- C5 pad 2: GND -> GNDA
- C6 pad 2: GND -> GNDA
- C7 pad 2: GND -> GNDPWR
- C8 pad 2: GND -> GNDPWR
- J1 pad 2: GND -> GNDPWR
- R1 pad 1: GND -> GNDPWR
- R11 pad 2: /SENSE_{U}+ -> /SENSE_{V}+
- R12 pad 2: GND -> GNDPWR
- R15 pad 1: /SENSE_{U} -> /SENSE_{V}
- R16 pad 2: /SENSE_{V}+ -> /SENSE_{U}+
- R17 pad 2: GND -> GNDPWR
- R20 pad 1: /SENSE_{V} -> /SENSE_{U}
- R22 pad 2: GND -> GNDPWR
- R3 pad 2: GND -> GNDPWR
- R4 pad 2: GND -> GNDPWR
- R5 pad 2: GND -> GNDPWR
- U1 pad 10: /~{USER_{INPUT}} -> /SPEED/ANGLE
- U1 pad 11: /ENABLE -> /~{USER_{INPUT}}
- U1 pad 12: /PWM_{V} -> /PWM_{U}
- U1 pad 14: /PWM_{U} -> /PWM_{V}
- U1 pad 9: /SPEED/ANGLE -> /ENABLE
- U2 pad 1: GND -> GNDPWR
- U2 pad 2: GND -> GNDPWR
- U2 pad 21: GND -> GNDPWR
- U2 pad 3: GND -> GNDPWR
- U2 pad 4: GND -> GNDPWR
- U2 pad 5: GND -> GNDPWR
- U2 pad 6: GND -> GNDPWR
- U2 pad 7: GND -> GNDPWR
- U2 pad 8: GND -> GNDPWR
- U4 pad 11: GND -> GNDA
Routing:
- net GNDPWR: track 0.00 -> 84.0 mm, vias 0 -> 27
- net /ENABLE: track 0.01 -> 53.2 mm, vias 0 -> 3
- net +3.3VA: track 0.00 -> 47.1 mm, vias 0 -> 6
- net /PWM_{V}: track 0.00 -> 42.4 mm, vias 0 -> 4
- net /PWM_{U}: track 0.00 -> 41.0 mm, vias 0 -> 4
- net /PWM_{W}: track 0.00 -> 35.9 mm, vias 0 -> 4
- net /SENSE_{W}+: track 0.00 -> 30.6 mm, vias 0 -> 2
- net /SENSE_{V}: track 0.00 -> 19.3 mm
- net /SENSE_{V}+: track 0.00 -> 16.9 mm, vias 0 -> 2
- net /SENSE_{U}+: track 0.00 -> 13.2 mm, vias 0 -> 2
- net /SENSE_{W}: track 0.00 -> 12.6 mm
- net /SENSE_{U}: track 0.00 -> 10.1 mm
- net GNDA: track 0.00 -> 9.21 mm, vias 0 -> 8
- net /NRST: track 0.00 -> 8.84 mm
- net /OSC_{IN}: track 0.00 -> 7.46 mm
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- added copper zone on In2.Cu, net +3V3
- added copper zone on In2.Cu, net /OUT_{U}
- added copper zone on In3.Cu, net /OUT_{U}
- added copper zone on In2.Cu, net /OUT_{V}
- added copper zone on In3.Cu, net /OUT_{V}
- added copper zone on In2.Cu, net /OUT_{W}
- added copper zone on In3.Cu, net /OUT_{W}
- added copper zone on F.Cu, net /SENSE_{U}+
- added copper zone on F.Cu, net /SENSE_{V}+
- added copper zone on F.Cu, net /SENSE_{W}+
- added copper zone on F.Cu, net /V_{pwrfuse}
- added copper zone on F.Cu, net /V_{pwr}
- added copper zone on In1.Cu, net GND
- added copper zone on In3.Cu, net GND
- added copper zone on In4.Cu, net GND
- added copper zone on In3.Cu, net GNDA
- added copper zone on B.Cu, net GNDPWR
- added copper zone on F.Cu, net GNDPWR
- added copper zone on In1.Cu, net GNDPWR
- added copper zone on In4.Cu, net GNDPWR

Commit message: 170323-v1.0
Parts:
- SW3: footprint Button_Switch_SMD:SW_SPST_B3U-1000P -> Button_Switch_SMD:SW_SPST_B3S-1000
- moved SW3 51.2 mm to (126.2, 115.6), turned to 180 degrees
- moved RV1 50.5 mm to (124.4, 108.9), turned to 90 degrees
- moved R9 44.8 mm to (129.7, 111.2), turned to 180 degrees
- moved R10 44.0 mm to (130.2, 109.7)
- moved C15 41.3 mm to (131.8, 109.2), turned to 0 degrees
- moved C14 10.9 mm to (132.5, 75.3), turned to 90 degrees
- moved R27 4.33 mm to (141.7, 91.1), turned to 180 degrees
- moved R26 1.18 mm to (146.9, 94.5), turned to -90 degrees
- moved J4 0.70 mm to (141.0, 117.5), turned to -90 degrees
Connections:
- C2 pad 2: GND -> GNDPWR
Routing:
- net /NRST: track 8.84 -> 55.0 mm, vias 0 -> 1
- net /I2C_{SCL}: track 0.00 -> 33.8 mm
- net /I2C_{SDA}: track 0.00 -> 32.6 mm, vias 0 -> 1
- net /SWD_{CLK}: track 0.00 -> 24.4 mm
- net /SWD_{IO}: track 0.00 -> 21.9 mm, vias 0 -> 1
- net /BOOT0_{SW}: track 2.85 -> 22.7 mm
- net /~{USER_{INPUT}}: track 0.00 -> 17.4 mm
- net /SPEED/ANGLE: track 0.00 -> 15.6 mm
- net +3V3: track 0.00 -> 14.0 mm, vias 0 -> 9
- net Net-(R10-Pad2): track 0.00 -> 11.2 mm
- net GND: track 6.29 -> 9.31 mm, vias 18 -> 16
- net +3.3VA: track 47.1 -> 49.4 mm
- net /OSC_{IN}: track 7.46 -> 9.34 mm
- net /OSC_{OUT}: track 2.48 -> 4.11 mm
- net Net-(D4-Pad1): track 0.00 -> 1.43 mm
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- added copper zone on F.Cu, net GNDA

Commit message: 190323
Routing:
- net GNDPWR: track 84.5 -> 85.2 mm
- net GNDA: vias 16 -> 17
- net GND: vias 16 -> 15
- added copper zone on B.Cu, net GNDA
- added copper zone on In1.Cu, net GNDA
- added copper zone on In4.Cu, net GNDA
