File: BLDC_driver_small.kicad_pcb (KiCad board)
At the start: 6 copper layers, 50 x 50 mm, 76 parts, among them J1 1x02 Terminal, J2 1x03 Terminal, J3 Conn_02x05_Odd_Even, J4 Conn_01x04, Q1 Q_PMOS_GDS, SW1 RST_SW, SW2 SW_SPDT, SW3 SW_Push_45deg, U1 STM32F030F4Px, U2 L6230Q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

Commit message: v190323-2
Parts:
- added NT1: NetTie_2, NetTie:NetTie-2_SMD_Pad2.0mm, F.Cu at (102.4, 107.5)
- added NT2: NetTie_2, NetTie:NetTie-2_SMD_Pad2.0mm, F.Cu at (120.5, 115.6)
- added NT3: NetTie_2, NetTie:NetTie-2_THT_Pad0.3mm, F.Cu at (119.9, 97.9)
- added NT4: NetTie_2, NetTie:NetTie-2_SMD_Pad0.5mm, F.Cu at (120.2, 91.5)
- added NT5: NetTie_2, NetTie:NetTie-2_SMD_Pad0.5mm, F.Cu at (116.8, 91.5)
- added NT6: NetTie_2, NetTie:NetTie-2_SMD_Pad0.5mm, F.Cu at (121.7, 72.2)
- moved R1 0.95 mm to (113.6, 110.5), turned to 90 degrees
Connections:
- J1 pad 2: GNDPWR -> GNDREF
- R1 pad 1: GNDPWR -> GNDREF
- R12 pad 2: GNDPWR -> /SENSE_{V}-
- R17 pad 2: GNDPWR -> /SENSE_{U}-
- R22 pad 2: GNDPWR -> /SENSE_{W}-
Routing:
- net GNDPWR: track 85.2 -> 3.48 mm, vias 27 -> 73
- net /SENSE_{W}-: track 0.00 -> 36.2 mm, vias 0 -> 2
- net /SENSE_{V}-: track 0.00 -> 25.1 mm, vias 0 -> 2
- net /SENSE_{U}-: track 0.00 -> 15.1 mm, vias 0 -> 2
- net GNDREF: track 0.00 -> 1.28 mm, vias 0 -> 9
- added copper zone on In2.Cu, net GNDPWR
- added copper zone on In3.Cu, net GNDPWR
- added copper zone on B.Cu, net GNDREF
- added copper zone on F.Cu, net GNDREF
- added copper zone on In1.Cu, net GNDREF
- added copper zone on In2.Cu, net GNDREF
- added copper zone on In3.Cu, net GNDREF
- added copper zone on In4.Cu, net GNDREF

Commit message: 200323-final
Parts:
- added NT7: NetTie_2, NetTie:NetTie-2_SMD_Pad0.5mm, F.Cu at (120.5, 98.5)
- added NT8: NetTie_2, NetTie:NetTie-2_SMD_Pad0.5mm, F.Cu at (120.5, 96.0)
- added NT9: NetTie_2, NetTie:NetTie-2_SMD_Pad0.5mm, F.Cu at (120.5, 97.2)
- added REF**: OSHW-Logo_5.7x6mm_SilkScreen, Symbol:OSHW-Logo_5.7x6mm_SilkScreen, F.Cu at (135.9, 103.7)
- added REF**: Fiducial_0.5mm_Mask1mm, Fiducial:Fiducial_0.5mm_Mask1mm, F.Cu at (116.1, 117.0)
- added REF**: Fiducial_0.5mm_Mask1mm, Fiducial:Fiducial_0.5mm_Mask1mm, F.Cu at (139.5, 109.9)
- added REF**: Fiducial_0.5mm_Mask1mm, Fiducial:Fiducial_0.5mm_Mask1mm, F.Cu at (113.1, 76.6)
- added REF**: Fiducial_0.5mm_Mask1mm, Fiducial:Fiducial_0.5mm_Mask1mm, F.Cu at (140.9, 79.1)
- added REF**: KiCad-Logo2_12mm_SilkScreen, Symbol:KiCad-Logo2_12mm_SilkScreen, B.Cu at (126.2, 106.4)
- added REF**: WEEE-Logo_4.2x6mm_SilkScreen, Symbol:WEEE-Logo_4.2x6mm_SilkScreen, B.Cu at (102.9, 105.7)
- added REF**: ESD-Logo_13.2x12mm_SilkScreen, Symbol:ESD-Logo_13.2x12mm_SilkScreen, B.Cu at (125.3, 90.4)
- added kibuzzard-6418180F: G***, kibuzzard-6418180F, F.Cu at (128.3, 74.7)
- added kibuzzard-64181824: G***, kibuzzard-64181824, F.Cu at (140.3, 77.4)
- added kibuzzard-641818A1: G***, kibuzzard-641818A1, F.Cu at (111.0, 116.5)
- added kibuzzard-6418190C: G***, kibuzzard-6418190C, F.Cu at (111.0, 112.9)
- added kibuzzard-64183623: G***, kibuzzard-64183623, F.Cu at (113.0, 88.1)
- added kibuzzard-6418363F: G***, kibuzzard-6418363F, F.Cu at (137.2, 114.8)
- added kibuzzard-64183651: G***, kibuzzard-64183651, F.Cu at (141.9, 106.6)
- added kibuzzard-64183661: G***, kibuzzard-64183661, F.Cu at (130.0, 107.2)
- added kibuzzard-64183696: G***, kibuzzard-64183696, F.Cu at (132.0, 113.9)
- added kibuzzard-641842DD: G***, kibuzzard-641842DD, F.Cu at (112.3, 72.1)
- added kibuzzard-641842EC: G***, kibuzzard-641842EC, F.Cu at (112.3, 70.7)
- added kibuzzard-64185F07: G***, kibuzzard-64185F07, B.Cu at (142.6, 76.2)
- NT3: footprint NetTie:NetTie-2_THT_Pad0.3mm -> NetTie:NetTie-2_SMD_Pad0.5mm
- moved NT3 2.03 mm to (120.5, 99.8), turned to 180 degrees
- moved NT5 0.05 mm to (116.9, 91.5)
Routing:
- net /ENABLE: track 53.2 -> 49.9 mm
- net /PWM_{U}: track 41.0 -> 41.9 mm
- net /PWM_{W}: track 35.9 -> 36.7 mm
- net GNDPWR: vias 73 -> 71
- net GNDA: vias 17 -> 24
- net GND: vias 15 -> 50
Other:
- board text added: "jlcjlcjlcjlc"

Commit message: v1.0
Parts:
- removed F1: Polyfuse, Fuse:Fuse_1206_3216Metric
- removed kibuzzard-64185F07: G***, kibuzzard-64185F07
- added kibuzzard-641877D0: G***, kibuzzard-641877D0, B.Cu at (142.1, 76.3)
- added kibuzzard-641879B1: G***, kibuzzard-641879B1, B.Cu at (127.2, 79.8)
- C1: footprint Capacitor_SMD:CP_Elec_10x12.5 -> Capacitor_SMD:CP_Elec_10x10.5
- C17, C18: value TBD -> 30p
Connections:
- Q1 pad 2: /V_{pwrfuse} -> /V_{pwr}
Routing:
- removed copper zone on F.Cu, net /V_{pwrfuse}
